Commit message: urdf_v2

File: leo_ws/src/leo/leo_description/urdf/new.urdf.xacro (robot description, xacro)
@@ -49,14 +49,12 @@
       </collision>
     </link>
+    <!--
+    <gazebo reference="wheel_${name}_link">
+      <mu1 value="10.0"/>
+      <mu2 value="10.0"/>
+    </gazebo>
+    -->
   </xacro:macro>
   <!-- LINKS -->
-  <!-- Used for fixing robot to Gazebo 'base_link' -->
-  <!-- <link name="world">
-    <origin xyz="0 0 0"/>
-  </link>
-  <joint name="fixed" type="floating">
-    <parent link="world"/>
-    <child link="base_link"/>
-  </joint> -->
   <link name="base_link">
     <inertial>
@@ -78,4 +76,32 @@
   </link>
   <link name="base_footprint"/>
+  <xacro:rocker_link name="L"/>
+  <xacro:rocker_link name="R"/>
+  <xacro:wheel_link name="FL" model="A"/>
+  <xacro:wheel_link name="RL" model="A"/>
+  <xacro:wheel_link name="FR" model="B"/>
+  <xacro:wheel_link name="RR" model="B"/>
+  <xacro:if value="$(arg default_antenna)">
+    <link name="antenna_link">
+      <inertial>
+        <mass value="0.001237"/>
+        <origin xyz="0 0 0.028828"/>
+        <inertia ixx="2.5529e-7" ixy="0.0" ixz="0.0" iyy="2.5529e-7" iyz="0.0" izz="1.354e-8"/>
+      </inertial>
+      <visual>
+        <geometry>
+          <mesh filename="package://leo_description/models/Antenna.dae"/>
+        </geometry>
+      </visual>
+      <collision>
+        <origin xyz="0 0 0.028"/>
+        <geometry>
+          <cylinder radius="0.0055" length="0.056"/>
+        </geometry>
+      </collision>
+    </link>
+  </xacro:if>
+  <link name="camera_frame"/>
+  <!-- JOINTS -->
   <xacro:if value="$(arg rockers_fixed)">
     <xacro:property name="rockers_joint_type" value="fixed"/>
@@ -101,5 +127,4 @@
       <child link="base_footprint"/>
   </joint>
-  <xacro:rocker_link name="L"/>
   <joint name="rocker_L_joint" type="${rockers_joint_type}">
     <origin xyz="0.00263 0.14167 -0.04731" rpy="0 0 ${pi}"/>
@@ -110,5 +135,4 @@
     <dynamics friction="0.1" damping="0.1"/> <!-- TODO -->
   </joint>
-  <xacro:rocker_link name="R"/>
   <joint name="rocker_R_joint" type="${rockers_joint_type}">
     <origin xyz="0.00263 -0.14167 -0.04731" rpy="0 0 0"/>
@@ -120,5 +144,4 @@
     <mimic joint="rocker_L_joint"/>
   </joint>
-  <xacro:wheel_link name="FL" model="A"/>
   <joint name="wheel_FL_joint" type="continuous">
     <origin xyz="-0.15256 -0.08214 -0.08802" rpy="0 0 0"/>
@@ -129,5 +152,4 @@
     <dynamics friction="0.1" damping="0.1"/> <!-- TODO -->
   </joint>
-  <xacro:wheel_link name="RL" model="A"/>
   <joint name="wheel_RL_joint" type="continuous">
     <origin xyz="0.15256 -0.08214 -0.08802" rpy="0 0 0"/>
@@ -138,5 +160,4 @@
     <dynamics friction="0.1" damping="0.1"/> <!-- TODO -->
   </joint>
-  <xacro:wheel_link name="FR" model="B"/>
   <joint name="wheel_FR_joint" type="continuous">
     <origin xyz="-0.15256 -0.08214 -0.08802" rpy="0 0 0"/>
@@ -147,5 +168,4 @@
     <dynamics friction="0.1" damping="0.1"/> <!-- TODO -->
   </joint>
-  <xacro:wheel_link name="RR" model="B"/>
   <joint name="wheel_RR_joint" type="continuous">
     <origin xyz="0.15256 -0.08214 -0.08802" rpy="0 0 0"/>
@@ -156,25 +176,4 @@
     <dynamics friction="0.1" damping="0.1"/> <!-- TODO -->
   </joint>
-  <xacro:if value="$(arg default_antenna)">
-    <link name="antenna_link">
-      <inertial>
-        <mass value="0.001237"/>
-        <origin xyz="0 0 0.028828"/>
-        <inertia ixx="2.5529e-7" ixy="0.0" ixz="0.0" iyy="2.5529e-7" iyz="0.0" izz="1.354e-8"/>
-      </inertial>
-      <visual>
-        <geometry>
-          <mesh filename="package://leo_description/models/Antenna.dae"/>
-        </geometry>
-      </visual>
-      <collision>
-        <origin xyz="0 0 0.028"/>
-        <geometry>
-          <cylinder radius="0.0055" length="0.056"/>
-        </geometry>
-      </collision>
-    </link>
-  </xacro:if>
-  <link name="camera_frame"/>
   <!-- TRANSMISSION -->
   <transmission name="wheel_FL_trans" type="SimpleTransmission">
